File: _autosave-First-Pcb-84Key-Design.kicad_pcb (KiCad board)
At the start: 2 copper layers, 24 parts, among them SW1 SW_Push, U1 ATmega32U4-AU, Y1 16Mhz

Commit message: Final 4 key
Parts:
- moved F1 4.05 mm to (-473.9, -326.0)
- moved R2 3.16 mm to (-467.5, -327.8)
- moved R3 3.16 mm to (-469.9, -327.8)
- moved C4 2.38 mm to (-464.3, -330.0)
- moved USB1 1.59 mm to (-469.1, -339.7)
Connections:
- R4 pad 1: Net-(R4-Pad1) -> GND
- U1 pad 33: Net-(U1-Pad33) -> Net-(R4-Pad2)
Routing:
- net +5V: track 167.6 -> 112.4 mm
- net Net-(USB1-Pad6): track 0.00 -> 16.3 mm
- net GND: track 107.0 -> 112.9 mm
- net D+: track 3.77 -> 8.51 mm
- net Net-(R1-Pad2): track 28.9 -> 33.5 mm
- net Net-(C3-Pad1): track 58.1 -> 53.7 mm, vias 0 -> 2
- net D-: track 3.76 -> 7.15 mm
- net VCC: track 6.34 -> 9.47 mm
- net Net-(R4-Pad2): track 32.6 -> 34.5 mm
- net Net-(R2-Pad1): track 12.3 -> 10.7 mm
- net Net-(R3-Pad1): track 14.1 -> 13.1 mm
- added copper zone on B.Cu, net GND
Other:
- rule trace_min: 0.2 -> 0
- board text added: "Rb4 V0.1"
