File: _autosave-First-Pcb-84Key-Design.sch (KiCad schematic (older format))
At the start: 24 parts, among them SW1 SW_Push, U1 ATmega32U4-AU, Y1 16Mhz

Commit message: Pertama Kelar
Connections:
- wire segments 69 -> 71
Changed lines of the file:
@@
 $EndComp
 Wire Wire Line
-	7650 3500 8200 3500
-Wire Wire Line
-	8400 3500 8800 3500
+	7650 3500 7850 3500
+Wire Wire Line
+	8400 3500 8450 3500
 $Comp
 L Device:R_Small R2
@@
 Text GLabel 2450 4150 1    50   Input ~ 0
 COL1
+Text GLabel 7650 1800 2    50   Input ~ 0
+COL1
+Text GLabel 7650 1900 2    50   Input ~ 0
+COL0
+Wire Wire Line
+	8150 3500 8200 3500
+Wire Wire Line
+	8550 3500 8800 3500
+Text GLabel 7650 2000 2    50   Input ~ 0
+ROW1
+Text GLabel 7650 3300 2    50   Input ~ 0
+ROW0
 $EndSCHEMATC

Commit message: Final 4 key
Connections:
- wire segments 71 -> 69
Changed lines of the file:
@@
 	1    0    0    -1
 $EndComp
-Wire Wire Line
-	7650 3500 7850 3500
-Wire Wire Line
-	8400 3500 8450 3500
 $Comp
 L Device:R_Small R2
@@
 Text GLabel 7650 1900 2    50   Input ~ 0
 COL0
-Wire Wire Line
-	8150 3500 8200 3500
-Wire Wire Line
-	8550 3500 8800 3500
 Text GLabel 7650 2000 2    50   Input ~ 0
 ROW1
 Text GLabel 7650 3300 2    50   Input ~ 0
 ROW0
+Wire Wire Line
+	7650 3500 8200 3500
+Wire Wire Line
+	8400 3500 8800 3500
 $EndSCHEMATC
